Commit message: Add location of meshes

File: urdf/bdx.urdf (robot description, URDF)
Before this commit: robot v3_bdx, 16 links, 15 joints
Links:
- link head_body_pitch: geometry collision mesh filename=package://bdx_description/meshes/head_body_pitch_collisions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; visual mesh filename=package://bdx_description/meshes/head_body_pitch_collisions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
- link head_body_roll: geometry collision mesh filename=package://bdx_description/meshes/head_body_roll_collisions.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; visual mesh filename=package://bdx_description/meshes/head_body_roll_collisions.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
- link head_body_yaw: geometry collision mesh filename=package://bdx_description/meshes/head_body_yaw_collisions.o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; visual mesh filename=package://bdx_description/meshes/head_body_yaw_collisions.o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
- link left_foot: geometry collision mesh filename=package://bdx_description/meshes/left_foot_collisions.obj; visual mesh filename=package://bdx_description/meshes/left_foot_collisions.obj
- link left_hip: geometry collision mesh filename=package://bdx_description/meshes/left_hip_collisions.obj; visual mesh filename=package://bdx_description/meshes/left_hip_collisions.obj
- link left_hip_rotation: geometry collision mesh filename=package://bdx_description/meshes/left_hip_rotation_collisio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; visual mesh filename=package://bdx_description/meshes/left_hip_rotation_collisio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
- link left_shin: geometry collision mesh filename=package://bdx_description/meshes/left_shin_collisions.obj; visual mesh filename=package://bdx_description/meshes/left_shin_collisions.obj
- link left_thigh: geometry collision mesh filename=package://bdx_description/meshes/left_thigh_collisions.obj; visual mesh filename=package://bdx_description/meshes/left_thigh_collisions.obj
- link neck: geometry collision mesh filename=package://bdx_description/meshes/neck_collisions.obj; visual mesh filename=package://bdx_description/meshes/neck_collisions.obj
- link right_foot: geometry collision mesh filename=package://bdx_description/meshes/right_foot_collisions.obj; visual mesh filename=package://bdx_description/meshes/right_foot_collisions.obj
- link right_hip: geometry collision mesh filename=package://bdx_description/meshes/right_hip_collisions.obj; visual mesh filename=package://bdx_description/meshes/right_hip_collisions.obj
- link right_hip_rotation: geometry collision mesh filename=package://bdx_description/meshes/right_hip_rotation_collisi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; visual mesh filename=package://bdx_description/meshes/right_hip_rotation_collisi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
- link right_shin: geometry collision mesh filename=package://bdx_description/meshes/right_shin_collisions.obj; visual mesh filename=package://bdx_description/meshes/right_shin_collisions.obj
- link right_thigh: geometry collision mesh filename=package://bdx_description/meshes/right_thigh_collisions.obj; visual mesh filename=package://bdx_description/meshes/right_thigh_collisions.obj
- link sw_bd0: geometry collision mesh filename=package://bdx_description/meshes/pelvis_collisions.obj; visual mesh filename=package://bdx_description/meshes/pelvis_collisions.obj
