Commit message: fix paths add dummy link

File: urdf/BD-XURDFJointsFixed.urdf (robot description, URDF)
Before this commit: robot BD-XURDFJointsFixed, 19 links, 18 joints
Links:
- added link base_link
- link body: geometry collision mesh filename=package://bdx_description/meshes/body.stl scale=0.001 0.001 0.001; visual mesh filename=package://bdx_description/meshes/body.stl scale=0.001 0.001 0.001
- link head: geometry collision mesh filename=package://bdx_description/meshes/head.stl scale=0.001 0.001 0.001; visual mesh filename=package://bdx_description/meshes/head.stl scale=0.001 0.001 0.001
- link left_antenna: geometry collision mesh filename=package://bdx_description/meshes/left_antenna.stl scale=0.001 0.001 0.001; visual mesh filename=package://bdx_description/meshes/left_antenna.stl scale=0.001 0.001 0.001
- link left_foot: geometry collision mesh filename=package://bdx_description/meshes/left_foot.stl scale=0.001 0.001 0.001; visual mesh filename=package://bdx_description/meshes/left_foot.stl scale=0.001 0.001 0.001
- link left_foot_pad: geometry collision mesh filename=package://bdx_description/meshes/left_foot_pad.stl scale=0.001 0.001 0.001; visual mesh filename=package://bdx_description/meshes/left_foot_pad.stl scale=0.001 0.001 0.001
- link left_hip: geometry collision mesh filename=package://bdx_description/meshes/left_hip.stl scale=0.001 0.001 0.001; visual mesh filename=package://bdx_description/meshes/left_hip.stl scale=0.001 0.001 0.001
- link left_hip_rotation: geometry collision mesh filename=package://bdx_description/meshes/left_hip_rotation.stl scale=0.001 0.001 0.001; visual mesh filename=package://bdx_description/meshes/left_hip_rotation.stl scale=0.001 0.001 0.001
- link left_lower_leg: geometry collision mesh filename=package://bdx_description/meshes/left_lower_leg.stl scale=0.001 0.001 0.001; visual mesh filename=package://bdx_description/meshes/left_lower_leg.stl scale=0.001 0.001 0.001
- link left_upper_leg: geometry collision mesh filename=package://bdx_description/meshes/left_upper_leg.stl scale=0.001 0.001 0.001; visual mesh filename=package://bdx_description/meshes/left_upper_leg.stl scale=0.001 0.001 0.001
- link neck_extension: geometry collision mesh filename=package://bdx_description/meshes/neck_extension.stl scale=0.001 0.001 0.001; visual mesh filename=package://bdx_description/meshes/neck_extension.stl scale=0.001 0.001 0.001
- link neck_pitch: geometry collision mesh filename=package://bdx_description/meshes/neck_pitch.stl scale=0.001 0.001 0.001; visual mesh filename=package://bdx_description/meshes/neck_pitch.stl scale=0.001 0.001 0.001
- link neck_yaw: geometry collision mesh filename=package://bdx_description/meshes/neck_yaw.stl scale=0.001 0.001 0.001; visual mesh filename=package://bdx_description/meshes/neck_yaw.stl scale=0.001 0.001 0.001
- link right_antenna: geometry collision mesh filename=package://bdx_description/meshes/right_antenna.stl scale=0.001 0.001 0.001; visual mesh filename=package://bdx_description/meshes/right_antenna.stl scale=0.001 0.001 0.001
- link right_foot: geometry collision mesh filename=package://bdx_description/meshes/right_foot.stl scale=0.001 0.001 0.001; visual mesh filename=package://bdx_description/meshes/right_foot.stl scale=0.001 0.001 0.001
- link right_foot_pad: geometry collision mesh filename=package://bdx_description/meshes/right_foot_pad.stl scale=0.001 0.001 0.001; visual mesh filename=package://bdx_description/meshes/right_foot_pad.stl scale=0.001 0.001 0.001
- link right_hip: geometry collision mesh filename=package://bdx_description/meshes/right_hip.stl scale=0.001 0.001 0.001; visual mesh filename=package://bdx_description/meshes/right_hip.stl scale=0.001 0.001 0.001
- link right_hip_rotation: geometry collision mesh filename=package://bdx_description/meshes/right_hip_rotation.stl scale=0.001 0.001 0.001; visual mesh filename=package://bdx_description/meshes/right_hip_rotation.stl scale=0.001 0.001 0.001
- link right_lower_leg: geometry collision mesh filename=package://bdx_description/meshes/right_lower_leg.stl scale=0.001 0.001 0.001; visual mesh filename=package://bdx_description/meshes/right_lower_leg.stl scale=0.001 0.001 0.001
- link right_upper_leg: geometry collision mesh filename=package://bdx_description/meshes/right_upper_leg.stl scale=0.001 0.001 0.001; visual mesh filename=package://bdx_description/meshes/right_upper_leg.stl scale=0.001 0.001 0.001
Joints:
- added joint fixed_base: type fixed, parent base_link, child body, origin xyz=0 0 0 rpy=0 0 0

File: urdf/BD-XURDFSimplifiedv2.urdf (robot description, URDF)
Before this commit: robot BD-XURDFSimplifiedv2, 19 links, 18 joints
Links:
- added link dummy_link
- link base_link: geometry collision mesh filename=package://bdx_description/meshes/base_link.stl scale=0.001 0.001 0.001; visual mesh filename=package://bdx_description/meshes/base_link.stl scale=0.001 0.001 0.001
- link head: geometry collision mesh filename=package://bdx_description/meshes/head.stl scale=0.001 0.001 0.001; visual mesh filename=package://bdx_description/meshes/head.stl scale=0.001 0.001 0.001
- link left_antenna: geometry collision mesh filename=package://bdx_description/meshes/left_antenna.stl scale=0.001 0.001 0.001; visual mesh filename=package://bdx_description/meshes/left_antenna.stl scale=0.001 0.001 0.001
- link left_foot: geometry collision mesh filename=package://bdx_description/meshes/left_foot.stl scale=0.001 0.001 0.001; visual mesh filename=package://bdx_description/meshes/left_foot.stl scale=0.001 0.001 0.001
- link left_foot_pad: geometry collision mesh filename=package://bdx_description/meshes/left_foot_pad.stl scale=0.001 0.001 0.001; visual mesh filename=package://bdx_description/meshes/left_foot_pad.stl scale=0.001 0.001 0.001
- link left_hip: geometry collision mesh filename=package://bdx_description/meshes/left_hip.stl scale=0.001 0.001 0.001; visual mesh filename=package://bdx_description/meshes/left_hip.stl scale=0.001 0.001 0.001
- link left_hip_rotation: geometry collision mesh filename=package://bdx_description/meshes/left_hip_rotation.stl scale=0.001 0.001 0.001; visual mesh filename=package://bdx_description/meshes/left_hip_rotation.stl scale=0.001 0.001 0.001
- link left_lower_leg: geometry collision mesh filename=package://bdx_description/meshes/left_lower_leg.stl scale=0.001 0.001 0.001; visual mesh filename=package://bdx_description/meshes/left_lower_leg.stl scale=0.001 0.001 0.001
- link left_upper_leg: geometry collision mesh filename=package://bdx_description/meshes/left_upper_leg.stl scale=0.001 0.001 0.001; visual mesh filename=package://bdx_description/meshes/left_upper_leg.stl scale=0.001 0.001 0.001
- link neck_extension: geometry collision mesh filename=package://bdx_description/meshes/neck_extension.stl scale=0.001 0.001 0.001; visual mesh filename=package://bdx_description/meshes/neck_extension.stl scale=0.001 0.001 0.001
- link neck_pitch: geometry collision mesh filename=package://bdx_description/meshes/neck_pitch.stl scale=0.001 0.001 0.001; visual mesh filename=package://bdx_description/meshes/neck_pitch.stl scale=0.001 0.001 0.001
- link neck_yaw: geometry collision mesh filename=package://bdx_description/meshes/neck_yaw.stl scale=0.001 0.001 0.001; visual mesh filename=package://bdx_description/meshes/neck_yaw.stl scale=0.001 0.001 0.001
- link right_antenna: geometry collision mesh filename=package://bdx_description/meshes/right_antenna.stl scale=0.001 0.001 0.001; visual mesh filename=package://bdx_description/meshes/right_antenna.stl scale=0.001 0.001 0.001
- link right_foot: geometry collision mesh filename=package://bdx_description/meshes/right_foot.stl scale=0.001 0.001 0.001; visual mesh filename=package://bdx_description/meshes/right_foot.stl scale=0.001 0.001 0.001
- link right_foot_pad: geometry collision mesh filename=package://bdx_description/meshes/right_foot_pad.stl scale=0.001 0.001 0.001; visual mesh filename=package://bdx_description/meshes/right_foot_pad.stl scale=0.001 0.001 0.001
- link right_hip: geometry collision mesh filename=package://bdx_description/meshes/right_hip.stl scale=0.001 0.001 0.001; visual mesh filename=package://bdx_description/meshes/right_hip.stl scale=0.001 0.001 0.001
- link right_hip_rotation: geometry collision mesh filename=package://bdx_description/meshes/right_hip_rotation.stl scale=0.001 0.001 0.001; visual mesh filename=package://bdx_description/meshes/right_hip_rotation.stl scale=0.001 0.001 0.001
- link right_lower_leg: geometry collision mesh filename=package://bdx_description/meshes/right_lower_leg.stl scale=0.001 0.001 0.001; visual mesh filename=package://bdx_description/meshes/right_lower_leg.stl scale=0.001 0.001 0.001
- link right_upper_leg: geometry collision mesh filename=package://bdx_description/meshes/right_upper_leg.stl scale=0.001 0.001 0.001; visual mesh filename=package://bdx_description/meshes/right_upper_leg.stl scale=0.001 0.001 0.001
Joints:
- added joint fixed_base: type fixed, parent dummy_link, child base_link, origin xyz=0 0 0 rpy=0 0 0

Commit message: change joint limits

File: urdf/BD-XURDFJointsFixed.urdf (robot description, URDF)
Before this commit: robot BD-XURDFJointsFixed, 20 links, 19 joints
Joints:
- joint head_pitch: limit lower=0.0 upper=0.0 effort=100.0 velocity=100.0 -> lower=-3.14159 upper=3.14159 effort=100.0 velocity=100.0
- joint head_roll: limit lower=0.0 upper=0.0 effort=100.0 velocity=100.0 -> lower=-3.14159 upper=3.14159 effort=100.0 velocity=100.0
- joint head_yaw: limit lower=0.0 upper=0.0 effort=100.0 velocity=100.0 -> lower=-3.14159 upper=3.14159 effort=100.0 velocity=100.0
- joint left_ankle: limit lower=0.0 upper=0.0 effort=100.0 velocity=100.0 -> lower=-3.14159 upper=3.14159 effort=100.0 velocity=100.0
- joint left_antenna: limit lower=0.0 upper=0.0 effort=100.0 velocity=100.0 -> lower=-3.14159 upper=3.14159 effort=100.0 velocity=100.0
- joint left_hip_pitch: limit lower=0.0 upper=0.0 effort=100.0 velocity=100.0 -> lower=-3.14159 upper=3.14159 effort=100.0 velocity=100.0
- joint left_hip_roll: limit lower=0.0 upper=0.0 effort=100.0 velocity=100.0 -> lower=-3.14159 upper=3.14159 effort=100.0 velocity=100.0
- joint left_hip_yaw: limit lower=0.0 upper=0.0 effort=100.0 velocity=100.0 -> lower=-3.14159 upper=3.14159 effort=100.0 velocity=100.0
- joint left_knee: limit lower=0.0 upper=0.0 effort=100.0 velocity=100.0 -> lower=-3.14159 upper=3.14159 effort=100.0 velocity=100.0
- joint neck_pitch: limit lower=0.0 upper=0.0 effort=100.0 velocity=100.0 -> lower=-3.14159 upper=3.14159 effort=100.0 velocity=100.0
- joint right_ankle: limit lower=0.0 upper=0.0 effort=100.0 velocity=100.0 -> lower=-3.14159 upper=3.14159 effort=100.0 velocity=100.0
- joint right_antenna: limit lower=0.0 upper=0.0 effort=100.0 velocity=100.0 -> lower=-3.14159 upper=3.14159 effort=100.0 velocity=100.0
- joint right_hip_pitch: limit lower=0.0 upper=0.0 effort=100.0 velocity=100.0 -> lower=-3.14159 upper=3.14159 effort=100.0 velocity=100.0
- joint right_hip_roll: limit lower=0.0 upper=0.0 effort=100.0 velocity=100.0 -> lower=-3.14159 upper=3.14159 effort=100.0 velocity=100.0
- joint right_hip_yaw: limit lower=0.0 upper=0.0 effort=100.0 velocity=100.0 -> lower=-3.14159 upper=3.14159 effort=100.0 velocity=100.0
- joint right_knee: limit lower=0.0 upper=0.0 effort=100.0 velocity=100.0 -> lower=-3.14159 upper=3.14159 effort=100.0 velocity=100.0
