Commit message: Update urdf

File: urdf/uki_bdx.urdf (robot description, URDF)
Before this commit: robot BD-XURDFJointsFixed, 23 links, 22 joints
Joints:
- joint neck_pitch: origin xyz=0.092558 -0.00375 0.053208 rpy=0 0 0 -> xyz=0.092558 -0.00375 0.053208 rpy=0 0.17 0

Commit message: Add Imu and Mavros to launch file

File: urdf/uki_bdx.urdf (robot description, URDF)
Before this commit: robot BD-XURDFJointsFixed, 23 links, 22 joints
Links:
- added link imu_link; visual box size=0.02 0.02 0.01
Joints:
- added joint imu_joint: type fixed, parent body, child imu_link, origin xyz=0 0 0.05 rpy=0 0 0

Commit message: add cameras to urdf

File: urdf/uki_bdx.urdf (robot description, URDF)
Before this commit: robot BD-XURDFJointsFixed, 24 links, 23 joints
Links:
- added link left_camera_frame; collision box size=0.032 0.032 0.032; visual box size=0.032 0.032 0.032
- added link right_camera_frame; collision box size=0.032 0.032 0.032; visual box size=0.032 0.032 0.032
Joints:
- added joint left_camera_frame_joint: type fixed, parent base_link, child left_camera_frame, origin xyz=0.14075 0.06 0.077 rpy=0 0 0
- added joint right_camera_frame_joint: type fixed, parent base_link, child right_camera_frame, origin xyz=0.14075 -0.06 0.077 rpy=0 0 0
